File: pcb/Ai_Cricket.sch (EAGLE design)
At the start: 34 parts, among them IC1 ATTINY45TINY85-SMT, IC2 TPS63002, J1 JST-2MM-MALE

Commit message: v1.0
Parts:
- removed LED1: (no value), Ai_LED:LED0603
- added L: YELLOW, Ai_LED:LED0603
- added ON: BLUE, Ai_LED:LED0603
- added R9: 300, Ai_Passives:RES0402
- added U$14: AI-LOGOXS, Ai_Miscellany:AI-LOGOXS
- D1: value (none) -> PMEG2010AEB; device microbuilder:DIODESOD-123 -> Ai_DiscreteSemis:DIODE-SCHOTTKYSOD-523
- D2, D3: value (none) -> BZT52; device Ai_DiscreteSemis:DIODE-ZENERBZT52 -> Ai_DiscreteSemis:DIODE-ZENER-BZT52
- D4: device diode:BAT54C -> Ai_DiscreteSemis:BAT54C
- F1: value (none) -> 1206L050YR
- IC1: value ATTINY45TINY85-SMT -> ATTINY85-SMT; device Ai_IC:ATTINY45TINY85-SMT -> Ai_IC:ATTINY85-SMT
- IC2: value TPS63002 -> TPS63000; device Alberto:TPS63002 -> Ai_Power:TPS63000
- J1: value JST-2MM-MALE -> JST-2-MALE; device Ai_Connectors:JST-2MM-MALE -> Ai_Connectors:JST-2-MALE
- R3: value 330 -> 1K
- renumbered @GND1 to GND7, @GND2 to GND8
Connections:
- new net N$1: L.A, R9.1
- net GND: now also L.C, ON.C; no longer LED1.C
- net N$4: now also ON.A; no longer LED1.A
- net PB0: now also R9.2
Other:
- note added: "GND"
- moved on the sheet: C1, C2, F1, R3, R6
