File: pcb/Ai_Cricket.brd (EAGLE design)
At the start: 30.6 x 30.6 mm, 34 parts, among them IC1 ATTINY45TINY85-SMT, IC2 TPS63002, J1 JST-2MM-MALE

Commit message: v1.0
Parts:
- removed LED1: (no value), Ai_LED:LED-0603
- added L: YELLOW, Ai_LED:LED-0603
- added ON: BLUE, Ai_LED:LED-0603
- added R9: 300, Ai_Passives:RES-0402
- added U$14: AI-LOGOXS, Ai_Miscellany:AI-LOGO-XS
- D1: value (none) -> PMEG2010AEB; device microbuilder:SOD-123 -> Ai_DiscreteSemis:SOD-523
- D2, D3: value (none) -> BZT52
- D4: device diode:SOT23 -> Ai_DiscreteSemis:SOT-23
- F1: value (none) -> 1206L050YR
- IC1: value ATTINY45TINY85-SMT -> ATTINY85-SMT
- IC2: value TPS63002 -> TPS63000; device Alberto:VFDFN-10 -> Ai_Power:10-VFDFN
- J1: value JST-2MM-MALE -> JST-2-MALE
- R3: value 330 -> 1K
- moved D1 5.41 mm to (21.1, 10.0)
- moved R8 4.92 mm to (17.9, 23.7), turned to 0 degrees
- moved R3 4.10 mm to (22.5, 14.6)
- moved R1 3.30 mm to (16.1, 21.7), turned to 90 degrees
- moved C2 2.55 mm to (13.3, 23.8), turned to 0 degrees
- moved D2 2.53 mm to (13.1, 21.4), turned to 270 degrees
- moved C3 2.29 mm to (17.8, 19.1)
- moved D3 1.88 mm to (17.7, 21.5), turned to 90 degrees
- moved R6 1.81 mm to (8.26, 12.8), turned to 90 degrees
- moved R5 1.78 mm to (6.99, 12.8)
- moved R7 1.78 mm to (5.71, 12.8)
- moved JS1 1.55 mm to (8.19, 10.1)
- moved F1 1.53 mm to (21.0, 20.2)
- moved C4 1.52 mm to (6.86, 18.0), turned to 90 degrees
- moved D4 1.25 mm to (10.7, 9.02)
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- renumbered @GND1 to GND7, @GND2 to GND8
Connections:
- removed net PAD1: J1.NC1
- removed net PAD2: J1.NC2
- new net N$1: L.A, R9.1
- net GND: now also L.C, ON.C; no longer LED1.C
- net N$4: now also ON.A; no longer LED1.A
- net PB0: now also R9.2
Routing:
- net GND: track 43.7 -> 3.71 mm, vias 6 -> 0
- net FB: track 10.3 -> 20.6 mm, vias 0 -> 2
- net N$6: track 1.83 -> 12.1 mm, vias 0 -> 2
- net VBUS: track 0.00 -> 7.77 mm
- net PB1: track 10.6 -> 16.4 mm
- net PB3: track 34.7 -> 29.0 mm, vias 3 -> 1
- net VPIN: track 0.00 -> 4.61 mm
- net VCC: track 44.2 -> 48.2 mm, vias 2 -> 4
- net PB2: track 10.1 -> 13.7 mm
- net N$10: track 9.36 -> 6.71 mm
- net N$1: track 0.00 -> 2.38 mm
- net PB0: track 13.7 -> 15.7 mm
- net VBAT: track 4.81 -> 2.86 mm
- net N$8: track 5.10 -> 6.87 mm
- net VIN: track 32.0 -> 33.6 mm, vias 0 -> 2
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- added copper zone on layer 1, net GND
Other:
- board text added: "CRICKET"
- board text added: "VPIN"
- board text added: "v1.0"
- board text added: "www.acrobotic.com"
- board text removed: "07-21-14"
- board text removed: "Cricket"
- board text removed: "Vin"

Commit message: updating and sending out to manufacture
Other:
- board size 30.6 x 30.6 mm -> 30.5 x 30.5 mm
Changed lines of the file:
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@@
 <setting verticaltext="up"/>
 </settings>
-<grid distance="5" unitdist="mil" unit="mil" style="lines" multiple="1" display="yes" altdistance="0.025" altunitdist="inch" altunit="inch"/>
+<grid distance="50" unitdist="mil" unit="mil" style="lines" multiple="1" display="yes" altdistance="0.025" altunitdist="inch" altunit="inch"/>
 <layers>
 <layer number="1" name="Top" color="4" fill="1" visible="yes" active="yes"/>
@@
 <board>
 <plain>
-<wire x1="0" y1="13.97" x2="30.48" y2="16.51" width="0" layer="20" curve="-180"/>
-<wire x1="30.48" y1="16.51" x2="0" y2="13.97" width="0" layer="20" curve="-180"/>
 <wire x1="2.06375" y1="15.24" x2="28.41625" y2="15.24" width="0" layer="51" curve="-180"/>
 <wire x1="28.41625" y1="15.24" x2="2.06375" y2="15.24" width="0" layer="51" curve="-180"/>
@@
 <text x="9.906" y="24.511" size="1.27" layer="22" ratio="15" rot="SMR150">0</text>
 <text x="19.177" y="20.193" size="1.27" layer="22" ratio="15" rot="MR0">CRICKET</text>
+<circle x="15.24" y="15.24" radius="15.24" width="0.0254" layer="20"/>
 </plain>
 <attributes>
